File: PCB_Designs/PulseFit.brd (EAGLE design)
At the start: 25.4 x 25.4 mm, 46 parts, among them IC1 TL072, IC2 TL072, IC3 TL072, IC4 TL072, Q1 PN2907A, Q2 2N2222A, Q3 PN2907A

Commit message: updates
Parts:
- removed JP1: (no value), SparkFun-Connectors:1X08_NO_SILK
- added BAT1, BAT2: 9V, SparkFun-Electromechanical:BATTCON_9V
- added BREAKOUT: (no value), SparkFun-Connectors:1X10_NO_SILK
- added C16, C17, C19, C20: 1u, resistor:C0402
- added C18: 10u, resistor:C0402
- added D2: 250mA/100V, SparkFun-DiscreteSemi:SOD-323
- added IC5: TL072, analog-devices:SO8
- added LED1: (no value), SparkFun-LED:LED-1206-BOTTOM
- added R14, R16, R17: 10k, resistor:R0402
- added R15: 1.5M, resistor:R0402
- C1: value 2.2u -> 4.2u
- IC1, IC2, IC3, IC4: device analog-devices:MSOP08 -> analog-devices:SO8
- R19: value 3.3M -> 4.3M
- moved R13 74.7 mm to (-33.3, -242.1)
Connections:
- removed net N$26: IC3.6, IC3.7
- removed net RECT: IC2.1, IC2.2, JP1.7, R11.2
- removed net SQU: IC4.1, JP1.5, R19.1, R20.1, R22.2
- removed net TRI: C1.1, IC1.3, JP1.4, Q1.3, Q3.2
- removed net TRI-FILT: C2.1, IC1.7, R6.2, R8.1
- new net COMP: BREAKOUT.10, IC5.7, R16.1
- new net FILTERED: BREAKOUT.4, C2.1, IC1.7, R6.2, R8.1
- new net MIXER: IC3.1, R12.1, R13.2
- new net N$12: IC5.1, IC5.2
- new net N$13: IC5.3, R17.2
- new net N$2: IC3.6, R13.1, R14.2
- new net PK: BREAKOUT.9, C18.2, D2.C, IC5.6, R15.1
- new net RECTIFIED: BREAKOUT.7, IC2.1, IC2.2, R11.2
- new net SAWTOOTH: C1.1, IC1.3, Q1.3, Q3.2
- new net SQUARE: BREAKOUT.5, IC4.1, R19.1, R20.1, R22.2
- new net VNEG: BAT2.-, C16.2, C18.1, C20.2, IC5.4, LED1.C, R15.2
- net GND: now also BAT1.-, BAT2.+, BREAKOUT.3, C16.1, C17.1, C19.1, C20.1, IC3.5, R17.1; no longer JP1.3, R13.2
- net N$10: now also LED1.A, R16.2; no longer IC3.5, R13.1
- net PULSE: now also BREAKOUT.8, D2.A, IC3.7, IC5.5, R14.1; no longer IC3.1, JP1.8, R12.1
- net SINE: now also BREAKOUT.6; no longer JP1.6
- net V_BATT: now also BAT1.+, C17.2, C19.2, IC5.8
- net V_NEG: now also BREAKOUT.2; no longer JP1.2
- net V_POS: now also BREAKOUT.1; no longer JP1.1
