File: PCB_Designs/PulseFit.sch (EAGLE design)
At the start: 46 parts, among them IC1 TL072, IC2 TL072, IC3 TL072, IC4 TL072, Q1 PN2907A, Q2 2N2222A, Q3 PN2907A

Commit message: schematic is finished, board needs more work
Parts:
- added BAT1, BAT2: 9V, SparkFun-Electromechanical:BATTERY9V
- added C16, C17: 1u, resistor:C-EUC0402
- added R14: 10k, resistor:R-US_R0402
Connections:
- net RECT renamed RECTIFIED
- net SQU renamed SQUARE
- removed net N$10: IC3B.IN+, R13.1
- removed net N$26: IC3B.IN-, IC3B.OUT
- removed net TRI: C1.1, IC1A.IN+, JP1.4, Q1.C, Q3.E
- removed net TRI-FILT: C2.1, IC1B.OUT, R6.2, R8.1
- new net FILTERED: C2.1, IC1B.OUT, JP1.4, R6.2, R8.1
- new net MIXER: IC3A.OUT, R12.1, R13.2
- new net N$2: IC3B.IN-, R13.1, R14.2
- new net SAWTOOTH: C1.1, IC1A.IN+, Q1.C, Q3.E
- new net VNEG: BAT2.-, C16.2
- net GND: now also BAT1.-, BAT2.+, C16.1, C17.1, IC3B.IN+; no longer R13.2
- net PULSE: now also IC3B.OUT, R14.1; no longer IC3A.OUT, R12.1
- net V_BATT: now also BAT1.+, C17.2
Other:
- note added: "Creative Commons License Attribution-NonCommercial- ShareAlike 3.0 Unported"
- note added: "Orlando S. Hoilett @oshoilett @CalvaryEngineer Made in the @IICEPD"
- note added: "PulseSim"
- note added: "Signal Mixer and PULSE Out"
- note removed: "Orlando S. Hoilett @CalvaryEngineer, @IICEPD PulseSim Creative Commons License Attribution-NonCommercial- ShareAlike 3.0 Unported"
- note removed: "Signal Mixer"
- note removed: "Unused terminated op amp"
- moved on the sheet: C10, C11, C12, C13, C14, C15, C2, C8, C9, IC1A, IC1B, IC1P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

Commit message: updates
Parts:
- removed JP1: (no value), SparkFun-Connectors:M08NO_SILK_FEMALE_PTH
- added BREAKOUT: M10NO_SILK_PTH_FEMALE, SparkFun-Connectors:M10NO_SILK_PTH_FEMALE
- added C18: 10u, resistor:C-EUC0402
- added C19, C20: 1u, resistor:C-EUC0402
- added D2: 250mA/100V, SparkFun-DiscreteSemi:DIODEBAS16
- added IC5: TL072, analog-devices:AD8607R
- added LED1: (no value), SparkFun-LED:LED1206-BOTTOM
- added R15: 1.5M, resistor:R-US_R0402
- added R16, R17: 10k, resistor:R-US_R0402
- C1: value 2.2u -> 4.2u
- IC1, IC2, IC3, IC4: device analog-devices:AD8607RM -> analog-devices:AD8607R
- R19: value 3.3M -> 4.3M
Connections:
- new net COMP: BREAKOUT.10, IC5B.OUT, R16.1
- new net N$10: LED1.A, R16.2
- new net N$12: IC5A.IN-, IC5A.OUT
- new net N$13: IC5A.IN+, R17.2
- new net PK: BREAKOUT.9, C18.2, D2.C, IC5B.IN-, R15.1
- net FILTERED: now also BREAKOUT.4; no longer JP1.4
- net GND: now also BREAKOUT.3, C19.1, C20.1, R17.1; no longer JP1.3
- net PULSE: now also BREAKOUT.8, D2.A, IC5B.IN+; no longer JP1.8
- net RECTIFIED: now also BREAKOUT.7; no longer JP1.7
- net SINE: now also BREAKOUT.6; no longer JP1.6
- net SQUARE: now also BREAKOUT.5; no longer JP1.5
- net VNEG: now also C18.1, C20.2, IC5P.V-, LED1.C, R15.2
- net V_BATT: now also C19.2, IC5P.V+
- net V_NEG: now also BREAKOUT.2; no longer JP1.2
- net V_POS: now also BREAKOUT.1; no longer JP1.1
Other:
- note added: ""Let's have a little fun and save the world while we're at it.""
- note added: "Comparator"
- note added: "Creative Commons License Attribution-NonCommercial- ShareAlike 4.0 Unported"
- note added: "From the admins at Learning about Electronics"
- note added: "LED Indicator"
- note added: "NOTE: This is not a medical device"
- note added: "Orlando S. Hoilett @oshoilett @CalvEngIO Made in the @IICEPDEng"
- note added: "Peak Detector"
- note added: "Sawtooth circuit from YouTuber w2aew."
- note added: "Unused terminated op amp"
- note removed: "Creative Commons License Attribution-NonCommercial- ShareAlike 3.0 Unported"
- note removed: "Orlando S. Hoilett @oshoilett @CalvaryEngineer Made in the @IICEPD"
- moved on the sheet: BAT1, BAT2, C16, C17
